File: hardware/kc87_pico_recorder.kicad_sch (KiCad schematic)
At the start: 18 parts, among them J1 DIN-5_180degree, U1 LM358

Commit message: wip: update schematic, R5 180 Ohm to 150 Ohm
Parts:
- R5: value 180 -> 150
Other:
- note added: "Einstellen des Pegels: Rechtecksignal 3,3V PP an PLAY_SIGNAL_PICO anlegen (Test-Firmware kc87_play_test oder Playback-Programm). PLAY_SIGNAL mit dem Oszilloskop messen und mit RV2 auf ca. 250mV PP einstellen (Bereich ca. 165 bis 250mV PP) (KC87-Eingang: Re = 10k, Ue_ss min. 24mV; Recorder-Norm min. 200mV). R4 + RV2 bilden zusammen mit R5 einen Spannungsteiler, die Quellimpedanz am KC87 betraegt m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"
- note removed: "Einstellen des Pegels: Rechtecksignal 3,3V PP an PLAY_SIGNAL_PICO anlegen (Test-Firmware kc87_play_test oder Playback-Programm). PLAY_SIGNAL mit dem Oszilloskop messen und mit RV2 auf ca. 250mV PP einstellen (Bereich ca. 200 bis 295mV PP) (KC87-Eingang: Re = 10k, Ue_ss min. 24mV; Recorder-Norm min. 200mV). R4 + RV2 bilden zusammen mit R5 einen Spannungsteiler, die Quellimpedanz am KC87 betraegt m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"
Changed lines of the file:
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@@
 		)
 	)
-	(text "Einstellen des Pegels: Rechtecksignal 3,3V PP an PLAY_SIGNAL_PICO anlegen (Test-Firmware kc87_play_test oder Playback-Programm).\nPLAY_SIGNAL mit dem Oszilloskop messen und mit RV2 auf ca. 250mV PP einstellen (Bereich ca. 200 bis 295mV PP)\n(KC87-Eingang: Re = 10k, Ue_ss min. 24mV; Recorder-Norm min. 200mV).\nR4 + RV2 bilden zusammen mit R5 einen Spannungsteiler, die Quellimpedanz am KC87 betraegt maximal ca. 180 Ohm."
+	(text "Einstellen des Pegels: Rechtecksignal 3,3V PP an PLAY_SIGNAL_PICO anlegen (Test-Firmware kc87_play_test oder Playback-Programm).\nPLAY_SIGNAL mit dem Oszilloskop messen und mit RV2 auf ca. 250mV PP einstellen (Bereich ca. 165 bis 250mV PP)\n(KC87-Eingang: Re = 10k, Ue_ss min. 24mV; Recorder-Norm min. 200mV).\nR4 + RV2 bilden zusammen mit R5 einen Spannungsteiler, die Quellimpedanz am KC87 betraegt maximal ca. 150 Ohm."
 		(exclude_from_sim no)
 		(at 21.844 139.7 0)
@@
 			)
 		)
-		(property "Value" "180"
+		(property "Value" "150"
 			(at 92.71 113.0299 0)
 			(show_name no)
